Commit message: Additional foot joint for biped robot with working training for linear velocity Need support for linear velocity in deployment Observation model input changed

File: resources/robots/go2_biped/urdf/go2.urdf (robot description, URDF)
Before this commit: robot go2_description, 29 links, 28 joints
Links:
- link RL_calf: mass 0.154 -> 0.654
- link RL_foot: mass 0.04 -> 0.10
- link RR_calf: mass 0.154 -> 0.654
- link RR_foot: mass 0.04 -> 0.10
Joints:
- joint RL_foot_joint: limit lower=-0.8 upper=0.8 effort=23.7 velocity=10.1 -> lower=-0.8 upper=0.8 effort=10.0 velocity=5.0
- joint RR_foot_joint: limit lower=-0.8 upper=0.8 effort=23.7 velocity=10.1 -> lower=-0.8 upper=0.8 effort=10.0 velocity=5.0

Commit message: Working training for biped with 2 actuators for feet

File: resources/robots/go2_biped/urdf/go2.urdf (robot description, URDF)
Before this commit: robot go2_description, 29 links, 28 joints
Joints:
- joint RL_foot_joint: limit lower=-0.8 upper=0.8 effort=10.0 velocity=5.0 -> lower=-0.3 upper=0.8 effort=10.0 velocity=5.0
- joint RR_foot_joint: limit lower=-0.8 upper=0.8 effort=10.0 velocity=5.0 -> lower=-0.3 upper=0.8 effort=10.0 velocity=5.0

Commit message: Working stable walking

File: resources/robots/go2_biped/urdf/go2.urdf (robot description, URDF)
Before this commit: robot go2_description, 29 links, 28 joints
Links:
- link RL_calf: mass 0.654 -> 0.154
- link RR_calf: mass 0.654 -> 0.154
Joints:
- joint RL_foot_joint: limit lower=-0.3 upper=0.8 effort=10.0 velocity=5.0 -> (none); origin xyz=0 0 -0.213 rpy=0 0 0 -> xyz=0 0 -0.213 rpy=0 0.5 0; type revolute -> fixed
- joint RR_foot_joint: limit lower=-0.3 upper=0.8 effort=10.0 velocity=5.0 -> (none); origin xyz=0 0 -0.213 rpy=0 0 0 -> xyz=0 0 -0.213 rpy=0 0.5 0; type revolute -> fixed
